File: HP21xxReceiverDriver.kicad_pcb (KiCad board)
At the start: 2 copper layers, 34.8 x 57.6 mm, 102 parts, among them J1 DIP24, J2 DIP24, J3 DIP24, Q1 MMBT2369A, Q10 MMBT2369A, Q11 MMBT2369A, Q12 MMBT2369A, Q13 MMBT2369A, Q14 MMBT2369A, Q15 MMBT2369A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

Commit message: Changed to 2k terminating resistors.
Parts:
- R16, R19, R22, R25, R28, R31, R34, R37, R40, R43, R46, R49, R5, R50, R51, R52, R53, R54: value 10k -> 2k
Changed lines of the file:
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@@
 			)
 		)
-		(property "Value" "10k"
+		(property "Value" "2k"
 			(at 0 1.17 90)
 			(layer "F.Fab")
@@
 			)
 		)
-		(property "LCSC" "C25744"
+		(property "LCSC" "C4109"
 			(at 0 0 270)
 			(unlocked yes)
@@
 			)
 		)
-		(pad "  " thru_hole rect
+		(pad "1" thru_hole rect
 			(at 0 0 90)
 			(size 1.7 1.7)
@@
 			)
 		)
-		(property "Value" "10k"
+		(property "Value" "2k"
 			(at 0 1.17 0)
 			(layer "F.Fab")
@@
 			)
 		)
-		(property "LCSC" "C25744"
+		(property "LCSC" "C4109"
 			(at 0 0 180)
 			(unlocked yes)
@@
 			)
 		)
-		(property "Value" "10k"
+		(property "Value" "2k"
 			(at 0 1.17 90)
 			(layer "F.Fab")
@@
 			)
 		)
-		(property "LCSC" "C25744"
+		(property "LCSC" "C4109"
 			(at 0 0 270)
 			(unlocked yes)
@@
 			)
 		)
-		(property "Value" "10k"
+		(property "Value" "2k"
 			(at 0 1.17 0)
 			(layer "F.Fab")
@@
 			)
 		)
-		(property "LCSC" "C25744"
+		(property "LCSC" "C4109"
 			(at 0 0 180)
 			(unlocked yes)
@@
 			)
 		)
-		(property "Value" "10k"
+		(property "Value" "2k"
 			(at 0 1.17 90)
 			(layer "F.Fab")
@@
 			)
 		)
-		(property "LCSC" "C25744"
+		(property "LCSC" "C4109"
 			(at 0 0 270)
 			(unlocked yes)
@@
 			)
 		)
-		(property "Value" "10k"
+		(property "Value" "2k"
 			(at 0 1.17 90)
 			(layer "F.Fab")
@@
 			)
 		)
-		(property "LCSC" "C25744"
+		(property "LCSC" "C4109"
 			(at 0 0 270)
 			(unlocked yes)
@@
 			)
 		)
-		(property "Value" "10k"
+		(property "Value" "2k"
 			(at 0 1.17 90)
 			(layer "F.Fab")
@@
 			)
 		)
-		(property "LCSC" "C25744"
+		(property "LCSC" "C4109"
 			(at 0 0 270)
 			(unlocked yes)
@@
 			)
 		)
-		(property "Value" "10k"
+		(property "Value" "2k"
 			(at 0 1.17 90)
 			(layer "F.Fab")
@@
 			)
 		)
-		(property "LCSC" "C25744"
+		(property "LCSC" "C4109"
 			(at 0 0 270)
 			(unlocked yes)
@@
 			)
 		)
-		(property "Value" "10k"
+		(property "Value" "2k"
 			(at 0 1.17 90)
 			(layer "F.Fab")
@@
 			)
 		)
-		(property "LCSC" "C25744"
+		(property "LCSC" "C4109"
 			(at 0 0 270)
 			(unlocked yes)
@@
 			)
 		)
-		(property "Value" "10k"
+		(property "Value" "2k"
 			(at 0 1.17 0)
 			(layer "F.Fab")
@@
 			)
 		)
-		(property "LCSC" "C25744"
+		(property "LCSC" "C4109"
 			(at 0 0 180)
 			(unlocked yes)
@@
 			)
 		)
-		(property "Value" "10k"
+		(property "Value" "2k"
 			(at 0 1.17 90)
 			(layer "F.Fab")
@@
 			)
 		)
-		(property "LCSC" "C25744"
+		(property "LCSC" "C4109"
 			(at 0 0 270)
 			(unlocked yes)
@@
 			)
 		)
-		(property "Value" "10k"
+		(property "Value" "2k"
 			(at 0 1.17 90)
 			(layer "F.Fab")
@@
 			)
 		)
-		(property "LCSC" "C25744"
+		(property "LCSC" "C4109"
 			(at 0 0 270)
 			(unlocked yes)
@@
 			)
 		)
-		(property "Value" "10k"
+		(property "Value" "2k"
 			(at 0 1.17 0)
 			(layer "F.Fab")
@@
 			)
 		)
-		(property "LCSC" "C25744"
+		(property "LCSC" "C4109"
 			(at 0 0 180)
 			(unlocked yes)
@@
 			)
 		)
-		(property "Value" "10k"
+		(property "Value" "2k"
 			(at 0 1.17 90)
 			(layer "F.Fab")
@@
 			)
 		)
-		(property "LCSC" "C25744"
+		(property "LCSC" "C4109"
 			(at 0 0 270)
 			(unlocked yes)
@@
 			)
 		)
-		(property "Value" "10k"
+		(property "Value" "2k"
 			(at 0 1.17 0)
 			(layer "F.Fab")
@@
 			)
 		)
-		(property "LCSC" "C25744"
+		(property "LCSC" "C4109"
 			(at 0 0 180)
 			(unlocked yes)
@@
 			)
 		)
-		(property "Value" "10k"
+		(property "Value" "2k"
 			(at 0 1.17 90)
 			(layer "F.Fab")
@@
 			)
 		)
-		(property "LCSC" "C25744"
+		(property "LCSC" "C4109"
 			(at 0 0 270)
 			(unlocked yes)
@@
 			)
 		)
-		(property "Value" "10k"
+		(property "Value" "2k"
 			(at 0 1.17 90)
 			(layer "F.Fab")
@@
 			)
 		)
-		(property "LCSC" "C25744"
+		(property "LCSC" "C4109"
 			(at 0 0 270)
 			(unlocked yes)
@@
 			)
 		)
-		(property "Value" "10k"
+		(property "Value" "2k"
 			(at 0 1.17 90)
 			(layer "F.Fab")
@@
 			)
 		)
-		(property "LCSC" "C25744"
+		(property "LCSC" "C4109"
 			(at 0 0 270)
 			(unlocked yes)
@@
 	)
 	(segment
-		(start 90.8304 74.5744)
-		(end 91.4146 74.5744)
+		(start 73.9394 84.8614)
+		(end 76.2 87.122)
 		(width 0.2)
 		(layer "F.Cu")
@@
 	)
 	(segment
-		(start 76.2 87.122)
-		(end 73.9394 84.8614)
+		(start 90.8304 74.5744)
+		(end 91.4146 74.5744)
 		(width 0.2)
 		(layer "F.Cu")
