File: HP21xxReceiverDriver.kicad_sch (KiCad schematic)
At the start: 102 parts, among them J1 DIP24, J2 DIP24, J3 DIP24, Q1 MMBT2369A, Q10 MMBT2369A, Q11 MMBT2369A, Q12 MMBT2369A, Q13 MMBT2369A, Q14 MMBT2369A, Q15 MMBT2369A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

Commit message: Changed to 2k terminating resistors.
Parts:
- R16, R19, R22, R25, R28, R31, R34, R37, R40, R43, R46, R49, R5, R50, R51, R52, R53, R54: value 10k -> 2k; LCSC C25744 -> C4109
Changed lines of the file:
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@@
 	)
 	(label "MINUS2VR1"
-		(at 236.22 36.83 0)
+		(at 234.95 36.83 0)
 		(effects
 			(font
@@
 			)
 		)
-		(property "Value" "10k"
+		(property "Value" "2k"
 			(at 111.76 133.3499 0)
 			(effects
@@
 			)
 		)
-		(property "LCSC" "C25744"
+		(property "LCSC" "C4109"
 			(at 109.22 132.08 0)
 			(effects
@@
 			)
 		)
-		(property "Value" "10k"
+		(property "Value" "2k"
 			(at 74.93 43.1799 0)
 			(effects
@@
 			)
 		)
-		(property "LCSC" "C25744"
+		(property "LCSC" "C4109"
 			(at 72.39 41.91 0)
 			(effects
@@
 			)
 		)
-		(property "Value" "10k"
+		(property "Value" "2k"
 			(at 17.78 33.0199 0)
 			(effects
@@
 			)
 		)
-		(property "LCSC" "C25744"
+		(property "LCSC" "C4109"
 			(at 20.32 31.75 0)
 			(effects
@@
 			)
 		)
-		(property "Value" "10k"
+		(property "Value" "2k"
 			(at 147.32 88.8999 0)
 			(effects
@@
 			)
 		)
-		(property "LCSC" "C25744"
+		(property "LCSC" "C4109"
 			(at 144.78 87.63 0)
 			(effects
@@
 			)
 		)
-		(property "Value" "10k"
+		(property "Value" "2k"
 			(at 147.32 133.3499 0)
 			(effects
@@
 			)
 		)
-		(property "LCSC" "C25744"
+		(property "LCSC" "C4109"
 			(at 144.78 132.08 0)
 			(effects
@@
 			)
 		)
-		(property "Value" "10k"
+		(property "Value" "2k"
 			(at 74.93 88.8999 0)
 			(effects
@@
 			)
 		)
-		(property "LCSC" "C25744"
+		(property "LCSC" "C4109"
 			(at 72.39 87.63 0)
 			(effects
@@
 			)
 		)
-		(property "Value" "10k"
+		(property "Value" "2k"
 			(at 111.76 88.8999 0)
 			(effects
@@
 			)
 		)
-		(property "LCSC" "C25744"
+		(property "LCSC" "C4109"
 			(at 109.22 87.63 0)
 			(effects
@@
 			)
 		)
-		(property "Value" "10k"
+		(property "Value" "2k"
 			(at 74.93 176.5299 0)
 			(effects
@@
 			)
 		)
-		(property "LCSC" "C25744"
+		(property "LCSC" "C4109"
 			(at 72.39 175.26 0)
 			(effects
@@
 			)
 		)
-		(property "Value" "10k"
+		(property "Value" "2k"
 			(at 111.76 176.5299 0)
 			(effects
@@
 			)
 		)
-		(property "LCSC" "C25744"
+		(property "LCSC" "C4109"
 			(at 109.22 175.26 0)
 			(effects
@@
 			)
 		)
-		(property "Value" "10k"
+		(property "Value" "2k"
 			(at 17.78 121.9199 0)
 			(effects
@@
 			)
 		)
-		(property "LCSC" "C25744"
+		(property "LCSC" "C4109"
 			(at 20.32 120.65 0)
 			(effects
@@
 			)
 		)
-		(property "Value" "10k"
+		(property "Value" "2k"
 			(at 17.78 62.2299 0)
 			(effects
@@
 			)
 		)
-		(property "LCSC" "C25744"
+		(property "LCSC" "C4109"
 			(at 20.32 60.96 0)
 			(effects
@@
 			)
 		)
-		(property "Value" "10k"
+		(property "Value" "2k"
 			(at 111.76 43.1799 0)
 			(effects
@@
 			)
 		)
-		(property "LCSC" "C25744"
+		(property "LCSC" "C4109"
 			(at 109.22 41.91 0)
 			(effects
@@
 			)
 		)
-		(property "Value" "10k"
+		(property "Value" "2k"
 			(at 147.32 177.7999 0)
 			(effects
@@
 			)
 		)
-		(property "LCSC" "C25744"
+		(property "LCSC" "C4109"
 			(at 144.78 176.53 0)
 			(effects
@@
 			)
 		)
-		(property "Value" "10k"
+		(property "Value" "2k"
 			(at 17.78 151.1299 0)
 			(effects
@@
 			)
 		)
-		(property "LCSC" "C25744"
+		(property "LCSC" "C4109"
 			(at 20.32 149.86 0)
 			(effects
@@
 			)
 		)
-		(property "Value" "10k"
+		(property "Value" "2k"
 			(at 147.32 43.1799 0)
 			(effects
@@
 			)
 		)
-		(property "LCSC" "C25744"
+		(property "LCSC" "C4109"
 			(at 144.78 41.91 0)
 			(effects
@@
 			)
 		)
-		(property "Value" "10k"
+		(property "Value" "2k"
 			(at 17.78 91.4399 0)
 			(effects
@@
 			)
 		)
-		(property "LCSC" "C25744"
+		(property "LCSC" "C4109"
 			(at 20.32 90.17 0)
 			(effects
@@
 			)
 		)
-		(property "Value" "10k"
+		(property "Value" "2k"
 			(at 74.93 133.3499 0)
 			(effects
@@
 			)
 		)
-		(property "LCSC" "C25744"
+		(property "LCSC" "C4109"
 			(at 72.39 132.08 0)
 			(effects
@@
 			)
 		)
-		(property "Value" "10k"
+		(property "Value" "2k"
 			(at 17.78 181.6099 0)
 			(effects
@@
 			)
 		)
-		(property "LCSC" "C25744"
+		(property "LCSC" "C4109"
 			(at 20.32 180.34 0)
 			(effects
