File: HP21xxReceiverDriver.kicad_sch (KiCad schematic)
At the start: 102 parts, among them J1 DIP24, J2 DIP24, J3 DIP24, Q1 MMBT2369A, Q10 MMBT2369A, Q11 MMBT2369A, Q12 MMBT2369A, Q13 MMBT2369A, Q14 MMBT2369A, Q15 MMBT2369A, Q16 MMBT2369A, Q17 MMBT2369A, Q18 MMBT2369A, Q2 MMBT2369A, Q3 MMBT2369A, Q4 MMBT2369A, Q5 MMBT2369A, Q6 MMBT2369A, Q7 MMBT2369A, Q8 MMBT2369A, Q9 MMBT2369A, U1 74ACT04, U2 AMS1117-3.3, U4 AMS1117-3.3

Commit message: Updated schematics and pcb for 3.3V pullups on the driver inputs.
Connections:
- net PLUS3V3R1: now also J3.13 (Pin_13)
- net PLUS3V3R2: now also J2.13 (Pin_13)
- net PLUS5D: no longer R49.1, R50.1, R51.1, R52.1, R53.1, R54.1
- net PLUS3_3V_IN: now reaches J1.1 (Pin_1)
- net PLUS3_3V_IN: now also R49.1, R50.1, R51.1, R52.1, R53.1, R54.1
- no-connect marks 28 -> 25
